Commit message: Narrow sim to robot-only: 4-wheel base + D555-style camera with built-in IMU
The Jetson owns mapping/nav (cuVSLAM/RTABMap, nvblox, Nav2) and the Pi5 owns
reasoning, so this repo drops everything that isn't the robot stand-in:

- delete rover_navigation, rover_localization, rover_docking and the nav
  launch/scripts; fleet_sim.sh now starts the sensors-only stack (MODE gone)
- remove the lidar and the body IMU; the camera macro grows a built-in IMU
  (/cam_1/imu, 200 Hz, cam_1_imu_optical_frame) mirroring realsense-ros
  unite_imu output
- pin GZ_PARTITION=rover_sim in launch scripts (a second gz instance on the
  machine otherwise steals the robot spawn) and narrow stop-script pkill
  patterns to this repo's processes only
- rewrite docs/INTERFACE.md as the fleet integration contract; update
  REAL_ROBOT_SWAP.md, README, CLAUDE.md

Verified: build clean, cam_1 topics at contract rates, no /scan//imu/data,
1 m drive via TwistStamped with odom+TF tracking, fleet_sim start/status/stop.

Co-Authored-By: Claude Fable 5 <noreply@anthropic.com>

File: rover_description/urdf/robots/rosmaster_x3.urdf.xacro (robot description, xacro)
@@ -8,6 +8,4 @@
     <xacro:include filename="$(find rover_description)/urdf/mech/mecanum_wheel.urdf.xacro"/>
     <xacro:include filename="$(find rover_description)/urdf/sensors/rgbd_camera.urdf.xacro"/>
-    <xacro:include filename="$(find rover_description)/urdf/sensors/lidar.urdf.xacro"/>
-    <xacro:include filename="$(find rover_description)/urdf/sensors/imu.urdf.xacro"/>
     <xacro:rosmaster_x3_base prefix="$(arg prefix)"/>
     <xacro:mecanum_wheel
@@ -31,6 +29,7 @@
       x_reflect="-1"
       y_reflect="-1"/>
-    <!-- 15 Hz / 8 m range: needed by depth-based mapping (nvblox) on the Jetson.
-         Defaults (2 Hz, 1.5 m) predate the perception integration. -->
+    <!-- The only exteroceptive sensor, mirroring the real rover: a RealSense
+         D555-style RGBD camera with its built-in IMU (topics /cam_1/*, /cam_1/imu).
+         15 Hz / 8 m range: needed by depth-based mapping (nvblox) on the Jetson. -->
     <xacro:rgbd_camera
       prefix="$(arg prefix)"
@@ -40,21 +39,4 @@
       update_rate="15"
       clip_far="8.0"/>
-    <xacro:lidar_sensor
-      prefix="$(arg prefix)"
-      parent="base_link"
-      frame_id="laser_frame"
-      xyz_offset="0 0 0.0825"
-      rpy_offset="0 0 0"
-      mesh_xyz_offset="0 0 0"
-      mesh_rpy_offset="${-M_PI/2} 0 0"
-      topic_name="scan"/>
-    <xacro:imu_sensor
-      prefix="$(arg prefix)"
-      parent="base_link"
-      frame_id="imu"
-      xyz_offset="0 0 0.006"
-      rpy_offset="0 0 0"
-      update_rate="15.0"
-      topic_name="imu/data"/>
     <xacro:include filename="$(find rover_description)/urdf/control/velocity_control_plugin.urdf.xacro" />
     <xacro:load_velocity_control_plugin use_gazebo="$(arg use_gazebo)"/>

File: rover_description/urdf/sensors/rgbd_camera.urdf.xacro (robot description, xacro)
@@ -43,4 +43,5 @@
     clip_far:=8.0
     update_rate:=15
+    imu_update_rate:=200
     always_on:=1
     visualize:=true
@@ -124,4 +125,19 @@
     </joint>
     <link name="${prefix}${camera_name}_color_optical_frame"/>
+    <!-- Built-in IMU, like the real RealSense D555. Frame layout mirrors
+         realsense-ros with unite_imu_method: data on <camera>/imu in
+         <camera>_imu_optical_frame. -->
+    <joint name="${prefix}${camera_name}_imu_joint" type="fixed">
+      <origin xyz="0 0 0" rpy="0 0 0" />
+      <parent link="${prefix}${camera_name}_link" />
+      <child link="${prefix}${camera_name}_imu_frame" />
+    </joint>
+    <link name="${prefix}${camera_name}_imu_frame"/>
+    <joint name="${prefix}${camera_name}_imu_optical_joint" type="fixed">
+      <origin xyz="${optical_xyz_offset}" rpy="${optical_rpy_offset}" />
+      <parent link="${prefix}${camera_name}_imu_frame" />
+      <child link="${prefix}${camera_name}_imu_optical_frame" />
+    </joint>
+    <link name="${prefix}${camera_name}_imu_optical_frame"/>
     <gazebo reference="${prefix}${camera_name}_link">
       <sensor name="${prefix}${camera_name}" type="rgbd_camera">
@@ -143,4 +159,17 @@
         <visualize>${visualize}</visualize>
       </sensor>
+      <!-- The camera's built-in IMU. Sensor pose rotates data into the
+           optical-frame axes (x right, y down, z forward), matching what
+           realsense-ros reports in <camera>_imu_optical_frame. Attached to
+           the camera link (not the massless imu frame links) so SDF joint
+           lumping keeps the sensor valid. -->
+      <sensor name="${prefix}${camera_name}_imu" type="imu">
+        <pose>0 0 0 ${-M_PI/2} 0 ${-M_PI/2}</pose>
+        <topic>${camera_name}/imu</topic>
+        <update_rate>${imu_update_rate}</update_rate>
+        <always_on>${always_on}</always_on>
+        <visualize>false</visualize>
+        <gz_frame_id>${prefix}${camera_name}_imu_optical_frame</gz_frame_id>
+      </sensor>
     </gazebo>
   </xacro:macro>
